Commit message: renamed resources folder

File: src/robot_properties_nyu_finger/resources/nyu_finger.urdf (robot description, URDF)
Before this commit: robot fingeredu, 6 links, 5 joints
Links:
- link finger_base_link: geometry collision mesh filename=package://meshes/base_back.stl scale=1 1 1; collision mesh filename=package://meshes/base_front.stl scale=1 1 1
- link finger_lower_link: geometry collision mesh filename=package://meshes/lower_link.stl scale=1 1 1; visual mesh filename=package://meshes/lower_link.stl scale=1 1 1
- link finger_middle_link: geometry collision mesh filename=package://meshes/middle_link.stl scale=1 1 1; visual mesh filename=package://meshes/middle_link.stl scale=1 1 1
- link finger_upper_link: geometry collision mesh filename=package://meshes/upper_link.stl scale=1 1 1; visual mesh filename=package://meshes/upper_link.stl scale=1 1 1

File: src/robot_properties_nyu_finger/resources/nyu_finger_double.urdf (robot description, URDF)
Before this commit: robot nyu_finger, 11 links, 10 joints
Links:
- link finger0_base_link: geometry collision mesh filename=package://meshes/base_back.stl scale=1 1 1; collision mesh filename=package://meshes/base_front.stl scale=1 1 1
- link finger0_lower_link: geometry collision mesh filename=package://meshes/lower_link.stl scale=1 1 1; visual mesh filename=package://meshes/lower_link.stl scale=1 1 1
- link finger0_middle_link: geometry collision mesh filename=package://meshes/middle_link.stl scale=1 1 1; visual mesh filename=package://meshes/middle_link.stl scale=1 1 1
- link finger0_upper_link: geometry collision mesh filename=package://meshes/upper_link.stl scale=1 1 1; visual mesh filename=package://meshes/upper_link.stl scale=1 1 1
- link finger1_base_link: geometry collision mesh filename=package://meshes/base_back.stl scale=1 1 1; collision mesh filename=package://meshes/base_front.stl scale=1 1 1
- link finger1_lower_link: geometry collision mesh filename=package://meshes/lower_link.stl scale=1 1 1; visual mesh filename=package://meshes/lower_link.stl scale=1 1 1
- link finger1_middle_link: geometry collision mesh filename=package://meshes/middle_link.stl scale=1 1 1; visual mesh filename=package://meshes/middle_link.stl scale=1 1 1
- link finger1_upper_link: geometry collision mesh filename=package://meshes/upper_link.stl scale=1 1 1; visual mesh filename=package://meshes/upper_link.stl scale=1 1 1
