Commit message: modfied the urdfs to reflect the mouting positions

File: src/robot_properties_nyu_finger/resources/nyu_finger_double.urdf (robot description, URDF)
Before this commit: robot nyu_finger, 11 links, 10 joints
Joints:
- joint base_to_finger0: origin xyz=-0.1 0 0.283 -> xyz=-0.0506 0 0.37
- joint base_to_finger1: origin xyz=0.1 0 0.283 rpy=0 0 3.14 -> xyz=0.0506 0 0.37 rpy=0 0 3.14
