Commit message: renamed config/urdf files and modified the wrapper to take a config object as an input

File: src/robot_properties_nyu_finger/resources/nyu_finger_double0.urdf (robot description, URDF)
Before this commit: robot nyu_finger1, 6 links, 5 joints
Links:
- removed link finger1_base_link
- removed link finger1_lower_link
- removed link finger1_middle_link
- removed link finger1_tip_link
- removed link finger1_upper_link
- added link finger0_base_link, mass 1; collision mesh filename=package://meshes/base_back.stl scale=1 1 1; collision mesh filename=package://meshes/base_front.stl scale=1 1 1
- added link finger0_lower_link, mass 0.03070; collision mesh filename=package://meshes/lower_link.stl scale=1 1 1; visual mesh filename=package://meshes/lower_link.stl scale=1 1 1
- added link finger0_middle_link, mass 0.14854; collision mesh filename=package://meshes/middle_link.stl scale=1 1 1; visual mesh filename=package://meshes/middle_link.stl scale=1 1 1
- added link finger0_tip_link, mass 0.01
- added link finger0_upper_link, mass 0.14854; collision mesh filename=package://meshes/upper_link.stl scale=1 1 1; visual mesh filename=package://meshes/upper_link.stl scale=1 1 1
Joints:
- removed joint base_to_finger1
- removed joint finger1_base_to_upper_joint
- removed joint finger1_lower_to_tip_joint
- removed joint finger1_middle_to_lower_joint
- removed joint finger1_upper_to_middle_joint
- added joint base_to_finger0: type fixed, parent base_link, child finger0_base_link, origin xyz=-0.0506 0 0.37
- added joint finger0_base_to_upper_joint: type revolute, parent finger0_base_link, child finger0_upper_link, origin xyz=0 0 0 rpy=0 0 0, axis -1 0 0, limit lower=-1.57079632679 upper=1.57079632679 effort=1000 velocity=1000
- added joint finger0_lower_to_tip_joint: type fixed, parent finger0_lower_link, child finger0_tip_link, origin xyz=0 -0.008 -0.16
- added joint finger0_middle_to_lower_joint: type revolute, parent finger0_middle_link, child finger0_lower_link, origin xyz=0 -0.03745 -0.16 rpy=0 0 0, axis 0 1 0, limit lower=-3.14159265359 upper=3.14159265359 effort=1000 velocity=1000
- added joint finger0_upper_to_middle_joint: type revolute, parent finger0_upper_link, child finger0_middle_link, origin xyz=0 -0.014 0 rpy=0 0 0, axis 0 1 0, limit lower=-1.57079632679 upper=1.57079632679 effort=1000 velocity=1000

File: src/robot_properties_nyu_finger/resources/nyu_finger_double1.urdf (robot description, URDF)
Before this commit: robot nyu_finger0, 6 links, 5 joints
Links:
- removed link finger0_base_link
- removed link finger0_lower_link
- removed link finger0_middle_link
- removed link finger0_tip_link
- removed link finger0_upper_link
- added link finger1_base_link, mass 1; collision mesh filename=package://meshes/base_back.stl scale=1 1 1; collision mesh filename=package://meshes/base_front.stl scale=1 1 1
- added link finger1_lower_link, mass 0.03070; collision mesh filename=package://meshes/lower_link.stl scale=1 1 1; visual mesh filename=package://meshes/lower_link.stl scale=1 1 1
- added link finger1_middle_link, mass 0.14854; collision mesh filename=package://meshes/middle_link.stl scale=1 1 1; visual mesh filename=package://meshes/middle_link.stl scale=1 1 1
- added link finger1_tip_link, mass 0.01
- added link finger1_upper_link, mass 0.14854; collision mesh filename=package://meshes/upper_link.stl scale=1 1 1; visual mesh filename=package://meshes/upper_link.stl scale=1 1 1
Joints:
- removed joint base_to_finger0
- removed joint finger0_base_to_upper_joint
- removed joint finger0_lower_to_tip_joint
- removed joint finger0_middle_to_lower_joint
- removed joint finger0_upper_to_middle_joint
- added joint base_to_finger1: type fixed, parent base_link, child finger1_base_link, origin xyz=0.0506 0 0.37 rpy=0 0 3.14
- added joint finger1_base_to_upper_joint: type revolute, parent finger1_base_link, child finger1_upper_link, origin xyz=0 0 0 rpy=0 0 0, axis -1 0 0, limit lower=-1.57079632679 upper=1.57079632679 effort=1000 velocity=1000
- added joint finger1_lower_to_tip_joint: type fixed, parent finger1_lower_link, child finger1_tip_link, origin xyz=0 -0.008 -0.16
- added joint finger1_middle_to_lower_joint: type revolute, parent finger1_middle_link, child finger1_lower_link, origin xyz=0 -0.03745 -0.16 rpy=0 0 0, axis 0 1 0, limit lower=-3.14159265359 upper=3.14159265359 effort=1000 velocity=1000
- added joint finger1_upper_to_middle_joint: type revolute, parent finger1_upper_link, child finger1_middle_link, origin xyz=0 -0.014 0 rpy=0 0 0, axis 0 1 0, limit lower=-1.57079632679 upper=1.57079632679 effort=1000 velocity=1000
